Commit message: Added simple 1dof robot for basic testing. Solved fitional force issue via removing adjacent collision meshes

File: data/robot/unitree-go1/urdf/go1.urdf (robot description, URDF)
Before this commit: robot go1_description, 23 links, 22 joints
Joints:
- joint FL_foot_fixed: axis (none) -> 0 0 1; limit (none) -> lower=-0.01 upper=0.01 effort=33.5 velocity=21; type fixed -> revolute
- joint RL_foot_fixed: axis (none) -> 0 0 1; limit (none) -> lower=-0.01 upper=0.01 effort=33.5 velocity=21; type fixed -> revolute
- joint RR_foot_fixed: axis (none) -> 0 0 1; limit (none) -> lower=-0.01 upper=0.01 effort=33.5 velocity=21; type fixed -> revolute
